Commit message: feat: separated components of torso and added color 	modified:   my_robot/urdf/my_robot.xacro

File: my_robot/urdf/my_robot.xacro (robot description, xacro)
@@ -1,5 +1,5 @@
 <?xml version='1.0'?>
 <robot name="my_robot" xmlns:xacro="http://www.ros.org/wiki/xacro">
-  <link name="chassis">
+  <link name="chassis_base">
     <pose>0 0 0.1 0 0 0</pose>
     <inertial>
@@ -12,5 +12,5 @@
       />
     </inertial>
-    <collision name="base_collision">
+    <collision name="chassis_base_collision">
       <origin xyz="0 0 0.1" rpy=" 0 0 0"/>
       <geometry>
@@ -18,5 +18,5 @@
       </geometry>
     </collision>
-    <visual name="base_visual">
+    <visual name="chassis_base_visual">
       <origin xyz="0 0 0.1" rpy=" 0 0 0"/>
       <geometry>
@@ -24,30 +24,73 @@
       </geometry>
     </visual>
-    <collision name="base_castor_block">
-      <origin xyz="0 0.21 0.05" rpy=" 0 0 0"/>
+  </link>
+  <link name="castor_block">
+    <inertial>
+      <mass value="0.5"/>
+      <origin xyz="0.0 0 0" rpy=" 0 0 0"/>
+      <inertia
+          ixx="0.1" ixy="0" ixz="0"
+          iyy="0.1" iyz="0"
+          izz="0.1"
+      />
+    </inertial>
+    <collision name="castor_block_collision">
+      <origin xyz="0 0 0" rpy=" 0 0 0"/>
       <geometry>
         <box size="0.08 0.15 .1"/>
       </geometry>
     </collision>
-    <visual name="base_castor_block">
-      <origin xyz="0 0.21 0.05" rpy=" 0 0 0"/>
+    <visual name="castor_block_visual">
+      <origin xyz="0 0 0" rpy=" 0 0 0"/>
       <geometry>
         <box size="0.08 0.15 .1"/>
       </geometry>
     </visual>
-    <collision name="body_collision">
-      <origin xyz="0 0 0.45" rpy=" 0 0 0"/>
+  </link>
+  <joint name="chassis_to_castor_block_joint" type="fixed">
+    <origin xyz="0.0 0.21 0.05" rpy="0.0 0.0 0.0"/>
+    <parent link="chassis_base"/>
+    <child link="castor_block"/>
+  </joint>
+  <link name="chassis_torso">
+    <inertial>
+      <mass value="2.5"/>
+      <origin xyz="0.0 0 0" rpy=" 0 0 0"/>
+      <inertia
+          ixx="0.1" ixy="0" ixz="0"
+          iyy="0.1" iyz="0"
+          izz="0.1"
+      />
+    </inertial>
+    <collision name="chassis_torso_collision">
+      <origin xyz="0 0 0.0" rpy=" 0 0 0"/>
       <geometry>
         <box size="0.35 0.25 0.5"/>
       </geometry>
     </collision>
-    <visual name="body_visual">
-      <origin xyz="0 0 0.45" rpy=" 0 0 0"/>
+    <visual name="chassis_torso_visual">
+      <origin xyz="0 0 0.0" rpy=" 0 0 0"/>
       <geometry>
         <box size="0.35 0.25 0.5"/>
       </geometry>
     </visual>
+  </link>
+  <joint name="torso_to_base" type="fixed">
+    <origin xyz="0.0 0.0 0.45" rpy="0.0 0.0 0.0"/>
+    <parent link="chassis_base"/>
+    <child link="chassis_torso"/>
+  </joint>
+  <link name="castor">
+    <inertial>
+      <mass value="0.05"/>
+      <origin xyz="0.0 0 0" rpy=" 0 0 0"/>
+      <inertia
+          ixx="0.1" ixy="0" ixz="0"
+          iyy="0.1" iyz="0"
+          izz="0.1"
+      />
+    </inertial>
     <visual name="caster_visual">
-      <origin xyz="0.0 0.225 -0.03" rpy="0.0 0.0 0.0"/>
+      <origin xyz="0.0 0.0 0.0" rpy="0.0 0.0 0.0"/>
       <geometry>
         <sphere radius="0.05"/>
@@ -58,5 +101,5 @@
     </visual>
     <collision name="caster_collision">
-      <origin xyz="0.0 0.225 -0.03" rpy="0.0 0.0 0.0"/>
+      <origin xyz="0.0 0.0 0.0" rpy="0.0 0.0 0.0"/>
       <geometry>
         <sphere radius="0.05"/>
@@ -64,4 +107,9 @@
     </collision>
   </link>
+  <joint name="castor_to_castor_block" type="fixed">
+    <origin xyz="0.0 0.0 -0.085" rpy="0.0 0.0 0.0"/>
+    <parent link="castor_block"/>
+    <child link="castor"/>
+  </joint>
   <link name="side_wheel_right">
     <inertial>
@@ -70,5 +118,5 @@
       <inertia ixx="0.01" ixy="0.0" ixz="0.0" iyy="0.01" iyz="0.0" izz="0.01"/>
     </inertial>
-    <visual name="side_wheel_visual">
+    <visual name="side_wheel_right_visual">
       <origin xyz="0 0 0" rpy="1.5707 0 1.5707"/>
       <geometry>
@@ -79,5 +127,5 @@
       </material>
     </visual>
-    <collision>
+    <collision name="side_wheel_right_collision">
       <origin xyz="0 0 0" rpy="1.5707 0 1.5707"/>
       <geometry>
@@ -88,5 +136,5 @@
   <joint name="right_wheel_hinge" type="continuous">
     <origin xyz="0.22 -0.1 0.06" rpy="0.0 0.0 0.0"/>
-    <parent link="chassis"/>
+    <parent link="chassis_base"/>
     <child link="side_wheel_right"/>
     <axis xyz="1 0 0"/>
@@ -100,5 +148,5 @@
       <inertia ixx="0.01" ixy="0.0" ixz="0.0" iyy="0.01" iyz="0.0" izz="0.01"/>
     </inertial>
-    <visual name="side_wheel_visual">
+    <visual name="side_wheel_left_visual">
       <origin xyz="0 0 0" rpy="1.5707 0 1.5707"/>
       <geometry>
@@ -109,5 +157,5 @@
       </material>
     </visual>
-    <collision>
+    <collision name="side_wheel_left_collision">
       <origin xyz="0 0 0" rpy="1.5707 0 1.5707"/>
       <geometry>
@@ -118,5 +166,5 @@
   <joint name="left_wheel_hinge" type="continuous">
     <origin xyz="-0.22 -0.1 0.06" rpy="0.0 0.0 0.0"/>
-    <parent link="chassis"/>
+    <parent link="chassis_base"/>
     <child link="side_wheel_left"/>
     <axis xyz="1 0 0"/>
@@ -148,6 +196,6 @@
 </link>
 <joint name="neck_joint" type="revolute">
-  <origin xyz="0.0 0.0 0.801" rpy="0.0 0.0 0.0"/>
-  <parent link="chassis"/>
+  <origin xyz="0.0 0.0 0.35" rpy="0.0 0.0 0.0"/>
+  <parent link="chassis_torso"/>
   <child link="head"/>
   <axis xyz="0 0 1"/>
@@ -155,15 +203,25 @@
   <dynamics damping="1.0" friction="1.0"/>
 </joint>
+<gazebo reference="chassis_base">
+  <material>Gazebo/Red</material>
+</gazebo>
+<gazebo reference="side_wheel_left">
+  <material>Gazebo/Green</material>
+</gazebo>
 <gazebo reference="side_wheel_right">
-  <material>Gazebo/BlueLaser</material>
-</gazebo>
-<gazebo reference="base_visual">
-  <material>Gazebo/Red</material>
-</gazebo>
-<gazebo reference="side_wheel_left">
-  <material>Gazebo/BlueLaser</material>
+  <material>Gazebo/Green</material>
+</gazebo>
+<gazebo reference="castor_block">
+  <material>Gazebo/Yellow</material>
+</gazebo>
+<gazebo reference="castor">
+  <material>Gazebo/Chrome</material>
+</gazebo>
+<gazebo reference="chassis_torso">
+  <material>Gazebo/Green</material>
 </gazebo>
 <gazebo reference="head">
-  <material>Gazebo/Yellow</material>
-</gazebo>
+  <material>Gazebo/Turquoise</material>
+</gazebo>
+chassis_torso
 </robot>

Commit message: feat: Added visual elements for Camera and Hokuyo lidar sensors

File: my_robot/urdf/my_robot.xacro (robot description, xacro)
@@ -66,5 +66,5 @@
       <origin xyz="0 0 0.0" rpy=" 0 0 0"/>
       <geometry>
-        <box size="0.35 0.25 0.5"/>
+        <box size="0.35 0.25 0.3"/>
       </geometry>
     </collision>
@@ -203,4 +203,55 @@
   <dynamics damping="1.0" friction="1.0"/>
 </joint>
+<link name="camera">
+  <inertial>
+    <origin xyz="0.0 0.0 0.0" rpy="0.0 0.0 0.0"/>
+    <mass value="0.1"/>
+    <inertia ixx="1e-6" ixy="0.0" ixz="0.0" iyy="1e-6" iyz="0.0" izz="1e-6"/>
+  </inertial>
+  <visual name="camera_visual">
+    <origin xyz="0.0 0.0 0.0" rpy="0.0 0.0 0.0"/>
+    <geometry>
+      <box size="0.05 0.05 0.05"/>
+    </geometry>
+  </visual>
+  <collision>
+    <origin xyz="0.0 0.0 0.0" rpy="0.0 0.0 0.0"/>
+    <geometry>
+      <box size="0.05 0.05 0.05"/>
+    </geometry>
+  </collision>
+</link>
+<joint name="camera_head" type="fixed">
+  <origin xyz="0.0 0.125 0.0" rpy="0.0 0.0 0.0"/>
+  <parent link="head"/>
+  <child link="camera"/>
+  <axis xyz="0.0 1 0.0"/>
+  <limit lower="0.0" upper="0.0" effort="0.0" velocity="0.0"/>
+</joint>
+<link name="hokuyo">
+  <inertial>
+    <origin xyz="0.0 0.0 0.0" rpy="0.0 0.0 0.0"/>
+    <mass value="1e-5"/>
+    <inertia ixx="1e-6" ixy="0.0" ixz="0.0" iyy="1e-6" iyz="0.0" izz="1e-6"/>
+  </inertial>
+  <visual name="hokuyo_visual">
+    <origin xyz="0.0 0.0 0.0" rpy="0.0 0.0 -1.5707"/>
+    <geometry>
+      <mesh filename="package://my_robot/meshes/hokuyo.dae"/>
+    </geometry>
+  </visual>
+  <collision>
+    <origin xyz="0.0 0.0 0.0" rpy="0.0 0.0 0.0"/>
+    <geometry>
+      <box size="0.1 0.1 0.1"/>
+    </geometry>
+  </collision>
+</link>
+<joint name="hokuyo_joint" type="fixed">
+  <origin xyz="0.0 0.0 0.13" rpy="0.0 0.0 0.0"/>
+  <parent link="head"/>
+  <child link="hokuyo"/>
+  <axis xyz="0.0 1 0.0"/>
+</joint>
 <gazebo reference="chassis_base">
   <material>Gazebo/Red</material>

Commit message: fix: Reduced the length of the torso so that the visual field of the camera includes the area close to the front castor wheel.

File: my_robot/urdf/my_robot.xacro (robot description, xacro)
@@ -72,10 +72,10 @@
       <origin xyz="0 0 0.0" rpy=" 0 0 0"/>
       <geometry>
-        <box size="0.35 0.25 0.5"/>
+        <box size="0.35 0.25 0.3"/>
       </geometry>
     </visual>
   </link>
   <joint name="torso_to_base" type="fixed">
-    <origin xyz="0.0 0.0 0.45" rpy="0.0 0.0 0.0"/>
+    <origin xyz="0.0 0.0 0.35" rpy="0.0 0.0 0.0"/>
     <parent link="chassis_base"/>
     <child link="chassis_torso"/>
@@ -196,5 +196,5 @@
 </link>
 <joint name="neck_joint" type="revolute">
-  <origin xyz="0.0 0.0 0.35" rpy="0.0 0.0 0.0"/>
+  <origin xyz="0.0 0.0 0.251" rpy="0.0 0.0 0.0"/>
   <parent link="chassis_torso"/>
   <child link="head"/>

Commit message: feat: Added sensor plugins for Camera, Hokoyu and differential drive controller
Also modified sizes of torso and head so as to allow clear field of view for
Lidar and adjusted camera angle to be able to see objects close to the robots
front area.

File: my_robot/urdf/my_robot.xacro (robot description, xacro)
@@ -1,4 +1,11 @@
 <?xml version='1.0'?>
 <robot name="my_robot" xmlns:xacro="http://www.ros.org/wiki/xacro">
+  <xacro:include filename="$(find my_robot)/urdf/my_robot.gazebo" />
+  <link name="robot_footprint"></link>
+  <joint name="robot_footprint_joint" type="fixed">
+    <origin xyz="0 0 0" rpy="0 0 0" />
+    <parent link="robot_footprint"/>
+    <child link="chassis_base" />
+  </joint>
   <link name="chassis_base">
     <pose>0 0 0.1 0 0 0</pose>
@@ -66,5 +73,5 @@
       <origin xyz="0 0 0.0" rpy=" 0 0 0"/>
       <geometry>
-        <box size="0.35 0.25 0.3"/>
+        <box size="0.33 0.22 0.25"/>
       </geometry>
     </collision>
@@ -72,10 +79,10 @@
       <origin xyz="0 0 0.0" rpy=" 0 0 0"/>
       <geometry>
-        <box size="0.35 0.25 0.3"/>
+        <box size="0.33 0.22 0.25"/>
       </geometry>
     </visual>
   </link>
   <joint name="torso_to_base" type="fixed">
-    <origin xyz="0.0 0.0 0.35" rpy="0.0 0.0 0.0"/>
+    <origin xyz="0.0 0.0 0.30" rpy="0.0 0.0 0.0"/>
     <parent link="chassis_base"/>
     <child link="chassis_torso"/>
@@ -185,5 +192,5 @@
     <origin xyz="0.0 0.0 0.0" rpy="0.0 0.0 0.0"/>
     <geometry>
-      <box size="0.35 0.25 0.2"/>
+      <box size="0.23 0.15 0.2"/>
     </geometry>
   </visual>
@@ -191,14 +198,14 @@
     <origin xyz="0.0 0.0 0.0" rpy="0.0 0.0 0.0"/>
     <geometry>
-      <box size="0.35 0.25 0.2"/>
+      <box size="0.23 0.15 0.2"/>
     </geometry>
   </collision>
 </link>
-<joint name="neck_joint" type="revolute">
-  <origin xyz="0.0 0.0 0.251" rpy="0.0 0.0 0.0"/>
+<joint name="neck_joint" type="continuous">
+  <origin xyz="0.0 0.0 0.201" rpy="0.0 0.0 0.0"/>
   <parent link="chassis_torso"/>
   <child link="head"/>
   <axis xyz="0 0 1"/>
-  <limit lower="-1.5707" upper="1.5707" effort="50.0" velocity="00.0"/>
+  <limit effort="100" velocity="100"/>
   <dynamics damping="1.0" friction="1.0"/>
 </joint>
@@ -222,9 +229,9 @@
   </collision>
 </link>
-<joint name="camera_head" type="fixed">
-  <origin xyz="0.0 0.125 0.0" rpy="0.0 0.0 0.0"/>
+<joint name="camera_head_joint" type="fixed">
+  <origin xyz="0.0 0.08 0.0" rpy="0.0 0.393 1.5707"/>
   <parent link="head"/>
   <child link="camera"/>
-  <axis xyz="0.0 1 0.0"/>
+  <axis xyz="0 0 0.0"/>
   <limit lower="0.0" upper="0.0" effort="0.0" velocity="0.0"/>
 </joint>
@@ -236,5 +243,5 @@
   </inertial>
   <visual name="hokuyo_visual">
-    <origin xyz="0.0 0.0 0.0" rpy="0.0 0.0 -1.5707"/>
+    <origin xyz="0.0 0.0 0.0" rpy="0.0 0.0 0.0"/>
     <geometry>
       <mesh filename="package://my_robot/meshes/hokuyo.dae"/>
@@ -249,5 +256,5 @@
 </link>
 <joint name="hokuyo_joint" type="fixed">
-  <origin xyz="0.0 0.0 0.13" rpy="0.0 0.0 0.0"/>
+  <origin xyz="0.0 0.04 0.13" rpy="0.0 0.0 1.5707"/>
   <parent link="head"/>
   <child link="hokuyo"/>

Commit message: feat: Placed the robot within the virtual world designed earlier

File: my_robot/urdf/my_robot.xacro (robot description, xacro)
@@ -145,6 +145,6 @@
     <parent link="chassis_base"/>
     <child link="side_wheel_right"/>
-    <axis xyz="1 0 0"/>
-    <limit effort="1000" velocity="1000"/>
+    <axis xyz="-1 0 0"/>
+    <limit effort="2000" velocity="2000"/>
     <dynamics damping="1.0" friction="1.0"/>
   </joint>
@@ -175,6 +175,6 @@
     <parent link="chassis_base"/>
     <child link="side_wheel_left"/>
-    <axis xyz="1 0 0"/>
-    <limit effort="1000" velocity="1000"/>
+    <axis xyz="-1 0 0"/>
+    <limit effort="2000" velocity="2000"/>
     <dynamics damping="1.0" friction="1.0"/>
   </joint>

Commit message: feat: Added the node drive_bot with a service to receive robot commands       for linear and angular movement.       Also made changes to the wheel radius and differential drive controller       params.

File: my_robot/urdf/my_robot.xacro (robot description, xacro)
@@ -14,8 +14,7 @@
       <origin xyz="0.0 0 0" rpy=" 0 0 0"/>
       <inertia
-          ixx="0.1" ixy="0" ixz="0"
-          iyy="0.1" iyz="0"
-          izz="0.1"
-      />
+          ixx="0.1" ixy="0"   ixz="0"
+                    iyy="0.1" iyz="0"
+                              izz="0.1"/>
     </inertial>
     <collision name="chassis_base_collision">
@@ -34,11 +33,10 @@
   <link name="castor_block">
     <inertial>
-      <mass value="0.5"/>
-      <origin xyz="0.0 0 0" rpy=" 0 0 0"/>
-      <inertia
-          ixx="0.1" ixy="0" ixz="0"
-          iyy="0.1" iyz="0"
-          izz="0.1"
-      />
+      <mass value="2.5"/>
+      <origin xyz="0.0 0 0" rpy=" 0 0 0"/>
+      <inertia
+          ixx="0.01" ixy="0"   ixz="0"
+                    iyy="0.01" iyz="0"
+                              izz="0.01"/>
     </inertial>
     <collision name="castor_block_collision">
@@ -62,11 +60,10 @@
   <link name="chassis_torso">
     <inertial>
-      <mass value="2.5"/>
-      <origin xyz="0.0 0 0" rpy=" 0 0 0"/>
-      <inertia
-          ixx="0.1" ixy="0" ixz="0"
-          iyy="0.1" iyz="0"
-          izz="0.1"
-      />
+      <mass value="1.0"/>
+      <origin xyz="0.0 0 0" rpy=" 0 0 0"/>
+      <inertia
+          ixx="0.1" ixy="0"   ixz="0"
+                    iyy="0.1" iyz="0"
+                              izz="0.1"/>
     </inertial>
     <collision name="chassis_torso_collision">
@@ -93,7 +90,7 @@
       <origin xyz="0.0 0 0" rpy=" 0 0 0"/>
       <inertia
-          ixx="0.1" ixy="0" ixz="0"
-          iyy="0.1" iyz="0"
-          izz="0.1"
+          ixx="0.1" ixy="0"   ixz="0"
+                    iyy="0.1" iyz="0"
+                              izz="0.1"
       />
     </inertial>
@@ -103,7 +100,4 @@
         <sphere radius="0.05"/>
       </geometry>
-      <material name="ball_material">
-        <color rgba="1.0 0.0 0.0 1.0"/>
-      </material>
     </visual>
     <collision name="caster_collision">
@@ -122,59 +116,57 @@
     <inertial>
       <origin xyz="0 0 0" rpy="1.5707 0 1.5707"/>
-      <mass value="0.5"/>
-      <inertia ixx="0.01" ixy="0.0" ixz="0.0" iyy="0.01" iyz="0.0" izz="0.01"/>
+      <mass value="5.0"/>
+      <inertia ixx="0.01" ixy="0.0"  ixz="0.0"
+                          iyy="0.01" iyz="0.0"
+                                     izz="0.01"/>
     </inertial>
     <visual name="side_wheel_right_visual">
       <origin xyz="0 0 0" rpy="1.5707 0 1.5707"/>
       <geometry>
-        <cylinder radius="0.15" length="0.02"/>
-      </geometry>
-      <material name="">
-        <color rgba="1.0 1.0 0.0 1.0"/>
-      </material>
+        <cylinder radius="0.1" length="0.02"/>
+      </geometry>
     </visual>
     <collision name="side_wheel_right_collision">
       <origin xyz="0 0 0" rpy="1.5707 0 1.5707"/>
       <geometry>
-        <cylinder radius="0.15" length="0.02"/>
+        <cylinder radius="0.1" length="0.02"/>
+      </geometry>
+    </collision>
+  </link>
+  <link name="side_wheel_left">
+    <inertial>
+      <origin xyz="0 0 0" rpy="1.5707 0 1.5707"/>
+      <mass value="5.0"/>
+      <inertia ixx="0.01" ixy="0.0"  ixz="0.0"
+                          iyy="0.01" iyz="0.0"
+                                    izz="0.01"/>
+    </inertial>
+    <visual name="side_wheel_left_visual">
+      <origin xyz="0 0 0" rpy="1.5707 0 1.5707"/>
+      <geometry>
+        <cylinder radius="0.1" length="0.02"/>
+      </geometry>
+    </visual>
+    <collision name="side_wheel_left_collision">
+      <origin xyz="0 0 0" rpy="1.5707 0 1.5707"/>
+      <geometry>
+        <cylinder radius="0.1" length="0.02"/>
       </geometry>
     </collision>
   </link>
   <joint name="right_wheel_hinge" type="continuous">
-    <origin xyz="0.22 -0.1 0.06" rpy="0.0 0.0 0.0"/>
+    <origin xyz="0.22 -0.1 0.01" rpy="0.0 0.0 0.0"/>
     <parent link="chassis_base"/>
     <child link="side_wheel_right"/>
     <axis xyz="-1 0 0"/>
-    <limit effort="2000" velocity="2000"/>
+    <limit effort="15000" velocity="2500"/>
     <dynamics damping="1.0" friction="1.0"/>
   </joint>
-  <link name="side_wheel_left">
-    <inertial>
-      <origin xyz="0 0 0" rpy="1.5707 0 1.5707"/>
-      <mass value="0.5"/>
-      <inertia ixx="0.01" ixy="0.0" ixz="0.0" iyy="0.01" iyz="0.0" izz="0.01"/>
-    </inertial>
-    <visual name="side_wheel_left_visual">
-      <origin xyz="0 0 0" rpy="1.5707 0 1.5707"/>
-      <geometry>
-        <cylinder radius="0.15" length="0.02"/>
-      </geometry>
-      <material name="">
-        <color rgba="1.0 1.0 0.0 1.0"/>
-      </material>
-    </visual>
-    <collision name="side_wheel_left_collision">
-      <origin xyz="0 0 0" rpy="1.5707 0 1.5707"/>
-      <geometry>
-        <cylinder radius="0.15" length="0.02"/>
-      </geometry>
-    </collision>
-  </link>
   <joint name="left_wheel_hinge" type="continuous">
-    <origin xyz="-0.22 -0.1 0.06" rpy="0.0 0.0 0.0"/>
+    <origin xyz="-0.22 -0.1 0.01" rpy="0.0 0.0 0.0"/>
     <parent link="chassis_base"/>
     <child link="side_wheel_left"/>
     <axis xyz="-1 0 0"/>
-    <limit effort="2000" velocity="2000"/>
+    <limit effort="15000" velocity="2500"/>
     <dynamics damping="1.0" friction="1.0"/>
   </joint>
@@ -182,10 +174,9 @@
   <inertial>
     <origin xyz="0.0 0.0 0.0" rpy="0.0 0.0 0.0"/>
-    <mass value="2.0"/>
+    <mass value="0.5"/>
     <inertia
-          ixx="0.05" ixy="0.05" ixz="0.05"
-          iyy="0.05" iyz="0.05"
-          izz="0.05"
-      />
+          ixx="1e-3" ixy="0.0"  ixz="0.0"
+                     iyy="1e-3" iyz="0.0"
+                                izz="1e-3"/>
   </inertial>
   <visual name="head_visual">
