Commit message: fix: Added a rear castor to fix balance issues. When the robot collides with      the ball or accellerates quickly it tips over backwards.

File: my_robot/urdf/my_robot.xacro (robot description, xacro)
@@ -31,5 +31,5 @@
     </visual>
   </link>
-  <link name="castor_block">
+  <link name="castor_block_front">
     <inertial>
       <mass value="2.5"/>
@@ -40,5 +40,5 @@
                               izz="0.01"/>
     </inertial>
-    <collision name="castor_block_collision">
+    <collision name="castor_block_front_collision">
       <origin xyz="0 0 0" rpy=" 0 0 0"/>
       <geometry>
@@ -46,5 +46,5 @@
       </geometry>
     </collision>
-    <visual name="castor_block_visual">
+    <visual name="castor_block_front_visual">
       <origin xyz="0 0 0" rpy=" 0 0 0"/>
       <geometry>
@@ -53,8 +53,35 @@
     </visual>
   </link>
-  <joint name="chassis_to_castor_block_joint" type="fixed">
+  <joint name="chassis_to_castor_block_front_joint" type="fixed">
     <origin xyz="0.0 0.21 0.05" rpy="0.0 0.0 0.0"/>
     <parent link="chassis_base"/>
-    <child link="castor_block"/>
+    <child link="castor_block_front"/>
+  </joint>
+  <link name="castor_block_back">
+    <inertial>
+      <mass value="2.5"/>
+      <origin xyz="0.0 0 0" rpy=" 0 0 0"/>
+      <inertia
+          ixx="0.01" ixy="0"   ixz="0"
+                    iyy="0.01" iyz="0"
+                              izz="0.01"/>
+    </inertial>
+    <collision name="castor_block_back_collision">
+      <origin xyz="0 0 0" rpy=" 0 0 0"/>
+      <geometry>
+        <box size="0.08 0.15 .1"/>
+      </geometry>
+    </collision>
+    <visual name="castor_block_back_visual">
+      <origin xyz="0 0 0" rpy=" 0 0 0"/>
+      <geometry>
+        <box size="0.08 0.15 .1"/>
+      </geometry>
+    </visual>
+  </link>
+  <joint name="chassis_to_castor_block_back_joint" type="fixed">
+    <origin xyz="0.0 -0.21 0.05" rpy="0.0 0.0 0.0"/>
+    <parent link="chassis_base"/>
+    <child link="castor_block_back"/>
   </joint>
   <link name="chassis_torso">
@@ -85,5 +112,5 @@
     <child link="chassis_torso"/>
   </joint>
-  <link name="castor">
+  <link name="castor_front">
     <inertial>
       <mass value="0.05"/>
@@ -95,5 +122,5 @@
       />
     </inertial>
-    <visual name="caster_visual">
+    <visual name="caster_front_visual">
       <origin xyz="0.0 0.0 0.0" rpy="0.0 0.0 0.0"/>
       <geometry>
@@ -101,5 +128,5 @@
       </geometry>
     </visual>
-    <collision name="caster_collision">
+    <collision name="caster_front_collision">
       <origin xyz="0.0 0.0 0.0" rpy="0.0 0.0 0.0"/>
       <geometry>
@@ -108,8 +135,36 @@
     </collision>
   </link>
-  <joint name="castor_to_castor_block" type="fixed">
-    <origin xyz="0.0 0.0 -0.085" rpy="0.0 0.0 0.0"/>
-    <parent link="castor_block"/>
-    <child link="castor"/>
+  <joint name="castor_to_castor_block_front" type="fixed">
+    <origin xyz="0.0 0.0 -0.09" rpy="0.0 0.0 0.0"/>
+    <parent link="castor_block_front"/>
+    <child link="castor_front"/>
+  </joint>
+  <link name="castor_back">
+    <inertial>
+      <mass value="0.05"/>
+      <origin xyz="0.0 0 0" rpy=" 0 0 0"/>
+      <inertia
+          ixx="0.1" ixy="0"   ixz="0"
+                    iyy="0.1" iyz="0"
+                              izz="0.1"
+      />
+    </inertial>
+    <visual name="caster_back_visual">
+      <origin xyz="0.0 0.0 0.0" rpy="0.0 0.0 0.0"/>
+      <geometry>
+        <sphere radius="0.05"/>
+      </geometry>
+    </visual>
+    <collision name="caster_back_collision">
+      <origin xyz="0.0 0.0 0.0" rpy="0.0 0.0 0.0"/>
+      <geometry>
+        <sphere radius="0.05"/>
+      </geometry>
+    </collision>
+  </link>
+  <joint name="castor_to_castor_block_back" type="fixed">
+    <origin xyz="0.0 0.0 -0.09" rpy="0.0 0.0 0.0"/>
+    <parent link="castor_block_back"/>
+    <child link="castor_back"/>
   </joint>
   <link name="side_wheel_right">
@@ -156,5 +211,5 @@
   </link>
   <joint name="right_wheel_hinge" type="continuous">
-    <origin xyz="0.22 -0.1 0.01" rpy="0.0 0.0 0.0"/>
+    <origin xyz="0.22 0.0 0.01" rpy="0.0 0.0 0.0"/>
     <parent link="chassis_base"/>
     <child link="side_wheel_right"/>
@@ -164,5 +219,5 @@
   </joint>
   <joint name="left_wheel_hinge" type="continuous">
-    <origin xyz="-0.22 -0.1 0.01" rpy="0.0 0.0 0.0"/>
+    <origin xyz="-0.22 0.0 0.01" rpy="0.0 0.0 0.0"/>
     <parent link="chassis_base"/>
     <child link="side_wheel_left"/>
@@ -261,5 +316,5 @@
   <material>Gazebo/Green</material>
 </gazebo>
-<gazebo reference="castor_block">
+<gazebo reference="castor_block_front">
   <material>Gazebo/Yellow</material>
 </gazebo>

Commit message: fix: Changes to neck joint to make this a fixed joint and small improvements in tracking

File: my_robot/urdf/my_robot.xacro (robot description, xacro)
@@ -248,11 +248,12 @@
   </collision>
 </link>
-<joint name="neck_joint" type="continuous">
+<!-- This is a fixed joint for now but I want to use this joint to make the head swivel in the future -->
+<joint name="neck_joint" type="fixed">
   <origin xyz="0.0 0.0 0.201" rpy="0.0 0.0 0.0"/>
   <parent link="chassis_torso"/>
   <child link="head"/>
   <axis xyz="0 0 1"/>
-  <limit effort="100" velocity="100"/>
-  <dynamics damping="1.0" friction="1.0"/>
+  <!--<limit effort="100" velocity="100"/>
+  <dynamics damping="1.0" friction="1.0"/>-->
 </joint>
 <link name="camera">

Commit message: fix: updated robot model to fix issue with amcl direction. updated params for tuning. The robot is now able to localise but path planning does not properly avoid objects.

File: my_robot/urdf/my_robot.xacro (robot description, xacro)
@@ -4,5 +4,5 @@
   <link name="robot_footprint"></link>
   <joint name="robot_footprint_joint" type="fixed">
-    <origin xyz="0 0 0" rpy="0 0 0" />
+    <origin xyz="0 0 0" rpy="0 0 -1.570796" />
     <parent link="robot_footprint"/>
     <child link="chassis_base" />
